File: HW/Monitor.sch (KiCad schematic (older format))
At the start: 22 parts, among them J1 TrigAndGnd, J2 Shunt1, J3 SD card header, J4 Shunt2, J5 Shunt3, J6 Barrel_Jack, U1 INA219AIDCNR, U2 BluePill_STM32F103C, U3 INA219AIDCNR, U4 INA219AIDCNR, U5 V7805-1000, U6 AMS117-3.3

Commit message: Layout and gerber
Parts:
- removed J1: TrigAndGnd, symbol Conn_01x02
- removed J2: Shunt1, symbol Conn_01x02
- removed J4: Shunt2, symbol Conn_01x02
- removed J5: Shunt3, symbol Conn_01x02
- removed U5: V7805-1000, digikey-footprints:3-SIP_Module_V7805-1000, symbol V7805-1000
- added J1: shunt 1 + 2, TerminalBlock_Phoenix:TerminalBlock_Phoenix_MPT-2.54mm_4pol, symbol Screw_Terminal_01x04
- added J2: Trig and shunt1, TerminalBlock_Phoenix:TerminalBlock_Phoenix_MPT-2.54mm_4pol, symbol Screw_Terminal_01x04
- added R4, R5: R, Resistors_SMD:R_0805_HandSoldering, symbol R
- added U5: OLED_128x32_i2c, Libs:OLED_128x32_I2C, symbol OLED_128x32_i2c
- added U7: LM2937, TO_SOT_Packages_SMD:SOT-223-3_TabPin2, symbol LM2937
- J3: footprint (none) -> Socket_Strips:Socket_Strip_Straight_1x07_Pitch2.54mm
- J6: footprint (none) -> Connectors:BARREL_JACK
- R1, R2, R3: footprint Resistors_SMD:R_0805_HandSoldering -> Resistors_SMD:R_2512_HandSoldering
- U2: footprint BluePill_breakouts:BluePill_STM32F103C -> Libs:BluePill_STM32F103C
Connections:
- net +12V: now also U7.1 (VIN)
- net +5V: now also J3.3 (Pin_3), U5.3 (VCC), U7.3 (VOUT)
- net GND: now also J2.4 (Pin_4), R5.2, U5.4 (GND), U7.2 (GND)
- net MISO: now also U2.13 (PB0)
- net NC: now also J3.1 (Pin_1); no longer J3.3 (Pin_3)
- net SCL: now also U5.2 (SCL)
- net SDA: now also U5.1 (SDA)
- net TRIG: now also J2.3 (Pin_3), R4.1; no longer U2.13 (PB0)
- net VCC: now also U2.40 (VCC3V3); no longer J3.1 (Pin_1)
- net at R1.1, U1.1 (IN+): now also J2.2 (Pin_2)
- net at R1.2, U1.2 (IN-): now also J2.1 (Pin_1)
- net at U2.25 (PA8): now also R4.2, R5.1
- net at R2.1, U3.1 (IN+): now also J1.4 (Pin_4)
- net at R2.2, U3.2 (IN-): now also J1.3 (Pin_3)
- net at R3.1, U4.1 (IN+): now also J1.2 (Pin_2)
- net at R3.2, U4.2 (IN-): now also J1.1 (Pin_1)
Other:
- moved on the sheet: C4, C5, J3, U2

Commit message: new version
Parts:
- removed J3: SD card header, Socket_Strips:Socket_Strip_Straight_1x07_Pitch2.54mm, symbol Conn_01x07_Female
- added BT1: Battery_Cell, Libs:Cheap_CR2032_holder, symbol Battery_Cell
- added C10: 10U, Capacitors_SMD:C_0805_HandSoldering, symbol C
- added C11, C12, C9: 100n, Capacitors_SMD:C_0805_HandSoldering, symbol C
- added C8: 1U, Capacitors_SMD:C_0805_HandSoldering, symbol C
- added J4: SD_Card, Connectors:SD_Card_Receptacle, symbol SD_Card
- added R6: 230R, Resistors_SMD:R_0805_HandSoldering, symbol R
- added U8: PC817, Libs:817opto, symbol PC817
- C1, C2, C3: value C -> 100n
- R4, R5: value R -> 1K
- U1, U3, U4: footprint digikey-footprints:SOT-23-8 -> TO_SOT_Packages_SMD:SOT-23-8_Handsoldering
Connections:
- net +5V: now also C11.1
- net CS: now also J4.1 (CD/DAT3)
- net GND: now also U2.14 (PB1), BT1.2 (-), C10.2, C11.2, C12.2, C8.2, C9.2, J4.12 (SHELL1), J4.13 (SHELL2), J4.3 (VSS), J4.6 (VSS), U8.2, U8.3; no longer R5.2
- net MISO: now also J4.7 (DAT0); no longer U2.13 (PB0)
- net MOSI: now also J4.2 (CMD)
- net SCK: now also J4.5 (CLK)
- net SCL: now also R4.2
- net SDA: now also R5.2
- net TRIG: now also U2.25 (PA8), U8.4; no longer J2.3 (Pin_3), R4.1
- net VCC: now also R4.1, R5.1, C10.1, C8.1, C9.1, J4.4 (VDD)
- net at U2.1 (VBAT): now also BT1.1 (+), C12.1
- new net: J2.3 (Pin_3), R6.2
- new net: R6.1, U8.1
Other:
- note added: "IF = 20mA\nVF = 1.2V"
- moved on the sheet: C2, J1, J2, R1, R2, R3, U1, U2, U3, U4
